Commit message: add navigation stack, simple navigator, configs, and .gitignore

File: src/eggy_robot_description/urdf/eggy_mecanum.urdf (robot description, URDF)
Before this commit: robot eggy_mecanum_robot, 4 links, 3 joints
Links:
- removed link laser_link
- added link laser_frame
Joints:
- joint base_to_imu: origin xyz=0 0 0.10 rpy=0 0 0 -> xyz=0.13 0 0.12 rpy=0 0 3.141592653589793
- joint base_to_laser: child laser_link -> laser_frame; origin xyz=0.12 0 0.16 rpy=0 0 0 -> xyz=0.05 0 0.28 rpy=0 0 0
